File: SpectrumAnayzerMini32.kicad_pcb (KiCad board)
At the start: 2 copper layers, 269.2 x 144.8 mm, 519 parts, among them J1 Input, J2 Output

Commit message: shrink the board
Parts:
- added J3: ST3, TerminalBlock_Phoenix:TerminalBlock_Phoenix_MPT-0,5-4-2.54_1x04_P2.54mm_Horizontal, B.Cu at (26.0, 60.3)
- J2: moved to F.Cu
- moved J1 316.7 mm to (27.3, 46.4)
- moved D1 314.9 mm to (40.0, 32.8)
- moved D10 314.9 mm to (40.0, 101.3)
- moved D11 314.9 mm to (40.0, 109.0)
- moved D12 314.9 mm to (40.0, 116.6)
- moved D13 314.9 mm to (40.0, 124.2)
- moved D14 314.9 mm to (40.0, 131.8)
- moved D15 314.9 mm to (40.0, 139.4)
- moved D16 314.9 mm to (40.0, 147.1)
- moved D2 314.9 mm to (40.0, 40.4)
- moved D3 314.9 mm to (40.0, 48.0)
- moved D4 314.9 mm to (40.0, 55.6)
- moved D5 314.9 mm to (40.0, 63.2)
- moved D6 314.9 mm to (40.0, 70.9)
- moved D7 314.9 mm to (40.0, 78.5)
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Connections:
- J1 pad 2: Net-(J1-Pad2) -> (no net)
- J2 pad 2: Net-(J2-Pad2) -> (no net)
Routing:
- net VDD: track 4411.6 -> 4293.4 mm, vias 95 -> 159
- net DIN: track 15.2 -> 54.4 mm
- net Net-(D512-Pad2): track 8.37 -> 17.4 mm, vias 0 -> 1
- net Net-(D448-Pad2): track 127.0 -> 120.3 mm
- net Net-(D384-Pad2): track 127.0 -> 120.3 mm
- net Net-(D112-Pad2): track 127.0 -> 120.3 mm
- net Net-(D128-Pad2): track 127.0 -> 120.3 mm
- net Net-(D80-Pad2): track 127.0 -> 120.3 mm
- net Net-(D64-Pad2): track 127.0 -> 120.3 mm
- net Net-(D48-Pad2): track 127.0 -> 120.3 mm
- net Net-(D400-Pad2): track 127.0 -> 120.3 mm
- net Net-(D336-Pad2): track 127.0 -> 120.3 mm
- net Net-(D32-Pad2): track 127.0 -> 120.3 mm
- net Net-(D288-Pad2): track 127.0 -> 120.3 mm
- net Net-(D256-Pad2): track 127.0 -> 120.3 mm
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Other:
- board size 269.2 x 144.8 mm -> 227.3 x 127 mm
- board text added: "+5v"
- board text added: "DIN"
- board text added: "DOUT"
- board text added: "GND"
- board text added: "PixelBlaze"
